Commit message: mbot_description

File: catkin_ws/src/mbot_description/urdf/mbot_with_camera.urdf (robot description, URDF)
Before this commit: robot mbot, 3 links, 2 joints
Links:
- added link back_caster_link; visual sphere radius=0.015
- added link camera_link; visual box size=0.03 0.04 0.04
- added link front_caster_link; visual sphere radius=0.015
Joints:
- added joint back_caster_joint: type continuous, parent base_link, child back_caster_link, origin xyz=-0.18 0 -0.095 rpy=0 0 0, axis 0 1 0
- added joint camera_joint: type fixed, parent base_link, child camera_link, origin xyz=0.17 0 0.10 rpy=0 0 0
- added joint front_caster_joint: type continuous, parent base_link, child front_caster_link, origin xyz=0.18 0 -0.095 rpy=0 0 0, axis 0 1 0

File: catkin_ws/src/mbot_description/urdf/mbot_with_kinect.urdf (robot description, URDF)
Before this commit: robot mbot, 3 links, 2 joints
Links:
- added link back_caster_link; visual sphere radius=0.015
- added link front_caster_link; visual sphere radius=0.015
- added link kinect_link; visual mesh filename=package://mbot_description/meshes/kinect.dae
Joints:
- added joint back_caster_joint: type continuous, parent base_link, child back_caster_link, origin xyz=-0.18 0 -0.095 rpy=0 0 0, axis 0 1 0
- added joint front_caster_joint: type continuous, parent base_link, child front_caster_link, origin xyz=0.18 0 -0.095 rpy=0 0 0, axis 0 1 0
- added joint kinect_joint: type fixed, parent base_link, child kinect_link, origin xyz=0.15 0 0.11 rpy=0 0 0

File: catkin_ws/src/mbot_description/urdf/mbot_with_laser.urdf (robot description, URDF)
Before this commit: robot mbot, 3 links, 2 joints
Links:
- added link back_caster_link; visual sphere radius=0.015
- added link front_caster_link; visual sphere radius=0.015
- added link laser_link; visual cylinder length=0.05 radius=0.05
Joints:
- added joint back_caster_joint: type continuous, parent base_link, child back_caster_link, origin xyz=-0.18 0 -0.095 rpy=0 0 0, axis 0 1 0
- added joint front_caster_joint: type continuous, parent base_link, child front_caster_link, origin xyz=0.18 0 -0.095 rpy=0 0 0, axis 0 1 0
- added joint laser_joint: type fixed, parent base_link, child laser_link, origin xyz=0 0 0.105 rpy=0 0 0
