Commit message: Finished Robot Model

File: catkin_ws/src/mbot_description/urdf/Jason_Robot.urdf (robot description, URDF)
Before this commit: robot Jason_Robot, 5 links, 4 joints
Links:
- added link front_castor_link; visual sphere radius=0.0165
- added link kinect_link; visual mesh filename=package://mbot_description/meshes/kinect.dae
Joints:
- added joint front_castor_joint: type continuous, parent base_link, child front_castor_link, origin xyz=0.1135 0 -0.0165 rpy=0 0 0, axis 0 1 0
- added joint kinect_joint: type fixed, parent base_link, child kinect_link, origin xyz=0.08 0 0.038 rpy=0 0 0
