Commit message: mbot_description

File: catkin_ws/src/mbot_description/urdf/mbot_base.urdf (robot description, URDF)
Before this commit: robot mbot, 3 links, 2 joints
Links:
- added link back_caster_link; visual sphere radius=0.015
- added link front_caster_link; visual sphere radius=0.015
Joints:
- added joint back_caster_joint: type continuous, parent base_link, child back_caster_link, origin xyz=-0.18 0 -0.095 rpy=0 0 0, axis 0 1 0
- added joint front_caster_joint: type continuous, parent base_link, child front_caster_link, origin xyz=0.18 0 -0.095 rpy=0 0 0, axis 0 1 0
