Commit message: new description

File: catkin_ws/src/mbot_description/urdf/mbot_base_gazebo.xacro (robot description, xacro)
@@ -1,112 +1,61 @@
 <?xml version="1.0"?>
-<robot name="mbot" xmlns:xacro="http://www.ros.org/wiki/xacro">
-    <!-- PROPERTY LIST -->
-    <xacro:property name="M_PI" value="3.1415926"/>
-    <xacro:property name="base_mass"   value="20" />
-    <xacro:property name="base_radius" value="0.20"/>
-    <xacro:property name="base_length" value="0.16"/>
-    <xacro:property name="wheel_mass"   value="2" />
-    <xacro:property name="wheel_radius" value="0.06"/>
-    <xacro:property name="wheel_length" value="0.025"/>
-    <xacro:property name="wheel_joint_y" value="0.19"/>
-    <xacro:property name="wheel_joint_z" value="0.05"/>
-    <xacro:property name="caster_mass"    value="0.5" />
-    <xacro:property name="caster_radius"  value="0.015"/> <!-- wheel_radius - ( base_length/2 - wheel_joint_z) -->
-    <xacro:property name="caster_joint_x" value="0.18"/>
-    <!-- Defining the colors used in this robot -->
-    <material name="yellow">
-        <color rgba="1 0.4 0 1"/>
-    </material>
-    <material name="black">
-        <color rgba="0 0 0 0.95"/>
-    </material>
-    <material name="gray">
-        <color rgba="0.75 0.75 0.75 1"/>
-    </material>
-    <!-- Macro for inertia matrix -->
-    <xacro:macro name="sphere_inertial_matrix" params="m r">
-        <inertial>
-            <mass value="${m}" />
-            <inertia ixx="${2*m*r*r/5}" ixy="0" ixz="0"
-                iyy="${2*m*r*r/5}" iyz="0"
-                izz="${2*m*r*r/5}" />
-        </inertial>
+<robot xmlns:xacro="http://www.ros.org/wiki/xacro">
+    <xacro:property name="M_PI" value="3.14159"/>
+    <xacro:property name="wheel_radius" value="0.033"/>
+    <xacro:property name="wheel_length" value="0.017"/>
+    <xacro:property name="base_link_radius" value="0.13"/>
+    <xacro:property name="base_link_length" value="0.005"/>
+    <xacro:property name="motor_radius" value="0.02"/>
+    <xacro:property name="motor_length" value="0.08"/>
+    <xacro:property name="motor_x" value="-0.055"/>
+    <xacro:property name="motor_y" value="0.075"/>
+    <xacro:property name="plate_height" value="0.07"/>
+    <xacro:property name="standoff_x" value="0.12"/>
+    <xacro:property name="standoff_y" value="0.10"/>
+    <!-- Define xacro:macro -->
+    <xacro:macro name="mrobot_standoff_2in" params="parent number x_loc y_loc z_loc">
+        <joint name="standoff_2in_${number}_joint" type="fixed">
+            <origin xyz="${x_loc} ${y_loc} ${z_loc}" rpy="0 0 0" />
+            <parent link="${parent}"/>
+            <child link="standoff_2in_${number}_link" />
+        </joint>
+        <link name="standoff_2in_${number}_link">
+            <inertial>
+                <mass value="0.001" />
+                <origin xyz="0 0 0" />
+                <inertia ixx="0.0001" ixy="0.0" ixz="0.0"
+                         iyy="0.0001" iyz="0.0"
+                         izz="0.0001" />
+            </inertial>
+            <visual>
+                <origin xyz=" 0 0 0 " rpy="0 0 0" />
+                <geometry>
+                    <box size="0.01 0.01 0.07" />
+                </geometry>
+                <material name="black">
+                    <color rgba="0.16 0.17 0.15 0.9"/>
+                </material>
+            </visual>
+            <collision>
+                <origin xyz="0.0 0.0 0.0" rpy="0 0 0" />
+                <geometry>
+                    <box size="0.01 0.01 0.07" />
+                </geometry>
+            </collision>
+        </link>
     </xacro:macro>
-    <xacro:macro name="cylinder_inertial_matrix" params="m r h">
-        <inertial>
-            <mass value="${m}" />
-            <inertia ixx="${m*(3*r*r+h*h)/12}" ixy = "0" ixz = "0"
-                iyy="${m*(3*r*r+h*h)/12}" iyz = "0"
-                izz="${m*r*r/2}" />
-        </inertial>
-    </xacro:macro>
-    <!-- Macro for robot wheel -->
-    <xacro:macro name="wheel" params="prefix reflect">
-        <joint name="${prefix}_wheel_joint" type="continuous">
-            <origin xyz="0 ${reflect*wheel_joint_y} ${-wheel_joint_z}" rpy="0 0 0"/>
-            <parent link="base_link"/>
-            <child link="${prefix}_wheel_link"/>
-            <axis xyz="0 1 0"/>
-        </joint>
-        <link name="${prefix}_wheel_link">
-            <visual>
-                <origin xyz="0 0 0" rpy="${M_PI/2} 0 0" />
-                <geometry>
-                    <cylinder radius="${wheel_radius}" length = "${wheel_length}"/>
-                </geometry>
-                <material name="gray" />
-            </visual>
-            <collision>
-                <origin xyz="0 0 0" rpy="${M_PI/2} 0 0" />
-                <geometry>
-                    <cylinder radius="${wheel_radius}" length = "${wheel_length}"/>
-                </geometry>
-            </collision>
-            <cylinder_inertial_matrix  m="${wheel_mass}" r="${wheel_radius}" h="${wheel_length}" />
-        </link>
-        <gazebo reference="${prefix}_wheel_link">
-            <material>Gazebo/Gray</material>
-        </gazebo>
-        <!-- Transmission is important to link the joints and the controller -->
-        <transmission name="${prefix}_wheel_joint_trans">
-            <type>transmission_interface/SimpleTransmission</type>
-            <joint name="${prefix}_wheel_joint" >
-                <hardwareInterface>hardware_interface/VelocityJointInterface</hardwareInterface>
-            </joint>
-            <actuator name="${prefix}_wheel_joint_motor">
-                <hardwareInterface>hardware_interface/VelocityJointInterface</hardwareInterface>
-                <mechanicalReduction>1</mechanicalReduction>
-            </actuator>
-        </transmission>
-    </xacro:macro>
-    <!-- Macro for robot caster -->
-    <xacro:macro name="caster" params="prefix reflect">
-        <joint name="${prefix}_caster_joint" type="continuous">
-            <origin xyz="${reflect*caster_joint_x} 0 ${-(base_length/2 + caster_radius)}" rpy="0 0 0"/>
-            <parent link="base_link"/>
-            <child link="${prefix}_caster_link"/>
-            <axis xyz="0 1 0"/>
-        </joint>
-        <link name="${prefix}_caster_link">
-            <visual>
-                <origin xyz="0 0 0" rpy="0 0 0"/>
-                <geometry>
-                    <sphere radius="${caster_radius}" />
-                </geometry>
-                <material name="black" />
-            </visual>
-            <collision>
-                <origin xyz="0 0 0" rpy="0 0 0"/>
-                <geometry>
-                    <sphere radius="${caster_radius}" />
-                </geometry>
-            </collision>
-            <sphere_inertial_matrix  m="${caster_mass}" r="${caster_radius}" />
-        </link>
-        <gazebo reference="${prefix}_caster_link">
-            <material>Gazebo/Black</material>
-        </gazebo>
-    </xacro:macro>
-    <xacro:macro name="mbot_base_gazebo">
+    <xacro:macro name="mrobot_body">
+        <material name="Green">
+            <color rgba="0.0 0.8 0.0 1.0"/>
+        </material>
+        <material name="yellow">
+            <color rgba="1 0.4 0 1"/>
+        </material>
+        <material name="black">
+            <color rgba="0 0 0 0.95"/>
+        </material>
+        <material name="gray">
+            <color rgba="0.75 0.75 0.75 1"/>
+        </material>
         <link name="base_footprint">
             <visual>
@@ -117,60 +66,226 @@
             </visual>
         </link>
-        <gazebo reference="base_footprint">
-            <turnGravityOff>false</turnGravityOff>
-        </gazebo>
+        <link name="base_link">
+            <inertial>
+                <mass value="2" />
+                <origin xyz="0 0 0.0" />
+                <inertia ixx="0.01" ixy="0.0" ixz="0.0"
+                         iyy="0.01" iyz="0.0" izz="0.5" />
+            </inertial>
+            <visual>
+                <origin xyz=" 0 0 0" rpy="0 0 0" />
+                <geometry>
+                    <cylinder length="${base_link_length}" radius="${base_link_radius}"/>
+                </geometry>
+                <material name="yellow" />
+            </visual>
+            <collision>
+                <origin xyz="0 0 0" rpy="0 0 0" />
+                <geometry>
+                    <cylinder length="${base_link_length}" radius="${base_link_radius}"/>
+                </geometry>
+            </collision>
+        </link>
         <joint name="base_footprint_joint" type="fixed">
-            <origin xyz="0 0 ${base_length/2 + caster_radius*2}" rpy="0 0 0" />
+            <origin xyz="0 0 ${wheel_radius}" rpy="0 0 0" />
             <parent link="base_footprint"/>
             <child link="base_link" />
         </joint>
-        <link name="base_link">
-            <visual>
-                <origin xyz=" 0 0 0" rpy="0 0 0" />
-                <geometry>
-                    <cylinder length="${base_length}" radius="${base_radius}"/>
+        <link name="left_motor">
+            <inertial>
+                <origin xyz="0.0 0 0"/>
+                <mass value="0.1" />
+                <inertia ixx="0.001" ixy="0.0" ixz="0.0"
+                         iyy="0.001" iyz="0.0" izz="0.001" />
+            </inertial>
+            <visual>
+                <origin xyz="0 0 0" rpy="${M_PI/2} 0 0" />
+                <geometry>
+                    <cylinder radius="${motor_radius}" length = "${motor_length}"/>
+                </geometry>
+                <material name="gray" />
+            </visual>
+            <collision>
+                <origin xyz="0 0 0" rpy="${M_PI/2} 0 0" />
+                <geometry>
+                    <cylinder radius="${motor_radius}" length = "${motor_length}"/>
+                </geometry>
+            </collision>
+        </link>
+        <joint name="base_left_motor_joint" type="fixed">
+            <origin xyz="${motor_x} ${motor_y} 0" rpy="0 0 0" />
+            <parent link="base_link"/>
+            <child link="left_motor" />
+        </joint>
+        <link name="left_wheel_link">
+            <inertial>
+                <origin xyz="0 0 0"/>
+                <mass value="0.01" />
+                <inertia ixx="0.001" ixy="0.0" ixz="0.0"
+                         iyy="0.001" iyz="0.0" izz="0.001" />
+            </inertial>
+            <visual>
+                <origin xyz="0 0 0" rpy="${M_PI/2} 0 0" />
+                <geometry>
+                    <cylinder radius="${wheel_radius}" length = "${wheel_length}"/>
+                </geometry>
+                <material name="white">
+                    <color rgba="1 1 1 0.9"/>
+                </material>
+            </visual>
+            <collision>
+                <origin xyz="0 0 0" rpy="${M_PI/2} 0 0" />
+                <geometry>
+                    <cylinder radius="${wheel_radius}" length = "${wheel_length}"/>
+                </geometry>
+            </collision>
+        </link>
+        <joint name="left_wheel_joint" type="continuous">
+            <origin xyz="0 ${(motor_length+wheel_length)/2} 0" rpy="0 0 0"/>
+            <parent link="left_motor"/>
+            <child link="left_wheel_link"/>
+            <axis xyz="0 1 0"/>
+        </joint>
+        <link name="right_motor">
+            <inertial>
+                <origin xyz="0.0 0 0"/>
+                <mass value="0.1" />
+                <inertia ixx="0.001" ixy="0.0" ixz="0.0"
+                         iyy="0.001" iyz="0.0" izz="0.001" />
+            </inertial>
+            <visual>
+                <origin xyz="0 0 0" rpy="${M_PI/2} 0 0" />
+                <geometry>
+                    <cylinder radius="${motor_radius}" length = "${motor_length}" />
+                </geometry>
+                <material name="gray" />
+            </visual>
+            <collision>
+                <origin xyz="0 0 0" rpy="${M_PI/2} 0 0" />
+                <geometry>
+                    <cylinder radius="${motor_radius}" length = "${motor_length}"/>
+                </geometry>
+            </collision>
+        </link>
+        <joint name="base_right_motor_joint" type="fixed">
+            <origin xyz="${motor_x} -${motor_y} 0" rpy="0 0 0" />
+            <parent link="base_link"/>
+            <child link="right_motor" />
+        </joint>
+        <link name="right_wheel_link">
+            <inertial>
+                <origin xyz="0 0 0"/>
+                <mass value="0.01" />
+                <inertia ixx="0.001" ixy="0.0" ixz="0.0"
+                         iyy="0.001" iyz="0.0" izz="0.001" />
+            </inertial>
+            <visual>
+                <origin xyz="0 0 0" rpy="${M_PI/2} 0 0" />
+                <geometry>
+                    <cylinder radius="${wheel_radius}" length = "${wheel_length}"/>
+                </geometry>
+                <material name="white">
+                    <color rgba="1 1 1 0.9"/>
+                </material>
+            </visual>
+            <collision>
+                <origin xyz="0 0 0" rpy="${M_PI/2} 0 0" />
+                <geometry>
+                    <cylinder radius="${wheel_radius}" length = "${wheel_length}"/>
+                </geometry>
+            </collision>
+        </link>
+        <joint name="right_wheel_joint" type="continuous">
+            <origin xyz="0 -${(motor_length+wheel_length)/2} 0" rpy="0 0 0"/>
+            <parent link="right_motor"/>
+            <child link="right_wheel_link"/>
+            <axis xyz="0 1 0"/>
+        </joint>
+        <link name="front_caster_link">
+            <inertial>
+                <origin xyz="0 0 0"/>
+                <mass value="0.001" />
+                <inertia ixx="0.0001" ixy="0.0" ixz="0.0"
+                         iyy="0.0001" iyz="0.0" izz="0.0001" />
+            </inertial>
+            <visual>
+                <origin xyz="0 0 0" rpy="${M_PI/2} 0 0"/>
+                <geometry>
+                    <sphere radius="${wheel_radius/2}" />
+                </geometry>
+                <material name="black" />
+            </visual>
+            <collision>
+                <origin xyz="0 0 0.01" rpy="${M_PI/2} 0 0" />
+                <geometry>
+                    <sphere radius="${wheel_radius/2}" />
+                </geometry>
+            </collision>
+        </link>
+        <joint name="front_caster_joint" type="fixed">
+            <origin xyz="${base_link_radius-wheel_radius/2} 0 -${wheel_radius/2}" rpy="0 0 0"/>
+            <parent link="base_link"/>
+            <child link="front_caster_link"/>
+        </joint>
+        <mrobot_standoff_2in parent="base_link" number="1" x_loc="-${standoff_x/2 + 0.03}" y_loc="-${standoff_y - 0.03}" z_loc="${plate_height/2}"/>
+        <mrobot_standoff_2in parent="base_link" number="2" x_loc="-${standoff_x/2 + 0.03}" y_loc="${standoff_y - 0.03}" z_loc="${plate_height/2}"/>
+        <mrobot_standoff_2in parent="base_link" number="3" x_loc="${standoff_x/2}" y_loc="-${standoff_y}" z_loc="${plate_height/2}"/>
+        <mrobot_standoff_2in parent="base_link" number="4" x_loc="${standoff_x/2}" y_loc="${standoff_y}" z_loc="${plate_height/2}"/>
+        <joint name="plate_1_joint" type="fixed">
+            <origin xyz="0 0 ${plate_height}" rpy="0 0 0" />
+            <parent link="base_link"/>
+            <child link="plate_1_link" />
+        </joint>
+        <link name="plate_1_link">
+            <inertial>
+                <mass value="0.1" />
+                <origin xyz="0 0 0" />
+                <inertia ixx="0.01" ixy="0.0" ixz="0.0"
+                         iyy="0.01" iyz="0.0" izz="0.01" />
+            </inertial>
+            <visual>
+                <origin xyz=" 0 0 0 " rpy="0 0 0" />
+                <geometry>
+                    <cylinder length="${base_link_length}" radius="${base_link_radius}"/>
+                </geometry>
+                <material name="yellow"/>
+            </visual>
+            <collision>
+                <origin xyz="0.0 0.0 0.0" rpy="0 0 0" />
+                <geometry>
+                    <cylinder length="${base_link_length}" radius="${base_link_radius}"/>
+                </geometry>
+            </collision>
+        </link>
+        <mrobot_standoff_2in parent="standoff_2in_1_link" number="5" x_loc="0" y_loc="0" z_loc="${plate_height}"/>
+        <mrobot_standoff_2in parent="standoff_2in_2_link" number="6" x_loc="0" y_loc="0" z_loc="${plate_height}"/>
+        <mrobot_standoff_2in parent="standoff_2in_3_link" number="7" x_loc="0" y_loc="0" z_loc="${plate_height}"/>
+        <mrobot_standoff_2in parent="standoff_2in_4_link" number="8" x_loc="0" y_loc="0" z_loc="${plate_height}"/>
+        <joint name="plate_2_joint" type="fixed">
+            <origin xyz="0 0 ${plate_height}" rpy="0 0 0" />
+            <parent link="plate_1_link"/>
+            <child link="plate_2_link" />
+        </joint>
+        <link name="plate_2_link">
+            <inertial>
+                <mass value="0.01" />
+                <origin xyz="0 0 0" />
+                <inertia ixx="0.001" ixy="0.0" ixz="0.0"
+                         iyy="0.001" iyz="0.0" izz="0.001" />
+            </inertial>
+            <visual>
+                <origin xyz=" 0 0 0 " rpy="0 0 0" />
+                <geometry>
+                    <cylinder length="${base_link_length}" radius="${base_link_radius}"/>
                 </geometry>
                 <material name="yellow" />
             </visual>
             <collision>
-                <origin xyz=" 0 0 0" rpy="0 0 0" />
-                <geometry>
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